Commit message: updated

File: dvrk_model/model/wsn_both_psms.urdf.xacro (robot description, xacro)
@@ -17,5 +17,5 @@
       <parent link="camera"/>
       <child link="right_camera_link"/>
-      <origin rpy="0.0 1.5708 1.5708" xyz="-0.005 0.0 0.5"/>
+      <origin rpy="0.0 1.5708 1.5708" xyz="-0.0028 0.0 0.5"/>
   </joint>
   <link name="right_camera_link">
@@ -37,5 +37,5 @@
       <parent link="camera"/>
       <child link="left_camera_link"/>
-      <origin rpy="0.0 1.5708 1.5708" xyz="0.005 0.00 0.5"/>
+      <origin rpy="0.0 1.5708 1.5708" xyz="0.0028 0.00 0.5"/>
   </joint>
   <link name="left_camera_link">
@@ -74,5 +74,5 @@
       <update_rate>30.0</update_rate>
       <camera name="right_camera">
-        <horizontal_fov>0.6</horizontal_fov>
+        <horizontal_fov>0.702</horizontal_fov>
         <image>
           <width>640</width>
@@ -114,5 +114,5 @@
       <update_rate>30.0</update_rate>
       <camera name="left_camera">
-        <horizontal_fov>0.6</horizontal_fov>
+        <horizontal_fov>0.702</horizontal_fov>
         <image>
           <width>640</width>
